File: CherryMX-RGB-THT/CherryMX-RGB-THT.kicad_pcb (KiCad board)
At the start: 2 copper layers, 17.8 x 17.8 mm, 5 parts, among them P1 CONN_01X07, SW1 SW_PUSH, U1 11AA010T

Commit message: Added the Option to use an SMD-LED on Backside
When using a single-color THT LED on the Front
Parts:
- added D3: LED, LEDs:LED_0805, B.Cu at (0.00, 3.17)
Routing:
- net /LED-3: track 4.58 -> 7.93 mm
- net /LED-2: track 11.8 -> 15.2 mm
Changed lines of the file:
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@@
 (kicad_pcb (version 4) (host pcbnew 4.0.1-stable)
   (general
-    (links 10)
+    (links 12)
     (no_connects 0)
-    (area -8.965001 -11.845 12.728334 10.6267)
+    (area -8.965001 -8.965001 8.965001 8.965001)
     (thickness 1.6)
     (drawings 4)
-    (tracks 18)
+    (tracks 25)
     (zones 0)
-    (modules 5)
+    (modules 6)
     (nets 9)
   )
@@
     )
   )
+  (module LEDs:LED_0805 (layer B.Cu)
+    (at 0 3.175)
+    (descr "LED 0805 smd package")
+    (tags "LED 0805 SMD")
+    (attr smd)
+    (fp_text reference D3 (at 3.175 0) (layer B.SilkS)
+      (effects (font (size 1 1) (thickness 0.15)) (justify mirror))
+    )
+    (fp_text value LED (at 0 -1.75) (layer B.Fab)
+      (effects (font (size 1 1) (thickness 0.15)) (justify mirror))
+    )
+    (fp_line (start -1.6 -0.75) (end 1.1 -0.75) (layer B.SilkS) (width 0.15))
+    (fp_line (start -1.6 0.75) (end 1.1 0.75) (layer B.SilkS) (width 0.15))
+    (fp_line (start -0.1 -0.15) (end -0.1 0.1) (layer B.SilkS) (width 0.15))
+    (fp_line (start -0.1 0.1) (end -0.25 -0.05) (layer B.SilkS) (width 0.15))
+    (fp_line (start -0.35 0.35) (end -0.35 -0.35) (layer B.SilkS) (width 0.15))
+    (fp_line (start 0 0) (end 0.35 0) (layer B.SilkS) (width 0.15))
+    (fp_line (start -0.35 0) (end 0 0.35) (layer B.SilkS) (width 0.15))
+    (fp_line (start 0 0.35) (end 0 -0.35) (layer B.SilkS) (width 0.15))
+    (fp_line (start 0 -0.35) (end -0.35 0) (layer B.SilkS) (width 0.15))
+    (fp_line (start 1.9 0.95) (end 1.9 -0.95) (layer B.CrtYd) (width 0.05))
+    (fp_line (start 1.9 -0.95) (end -1.9 -0.95) (layer B.CrtYd) (width 0.05))
+    (fp_line (start -1.9 -0.95) (end -1.9 0.95) (layer B.CrtYd) (width 0.05))
+    (fp_line (start -1.9 0.95) (end 1.9 0.95) (layer B.CrtYd) (width 0.05))
+    (pad 2 smd rect (at 1.04902 0 180) (size 1.19888 1.19888) (layers B.Cu B.Paste B.Mask)
+      (net 5 /LED-3))
+    (pad 1 smd rect (at -1.04902 0 180) (size 1.19888 1.19888) (layers B.Cu B.Paste B.Mask)
+      (net 6 /LED-2))
+    (model LEDs.3dshapes/LED_0805.wrl
+      (at (xyz 0 0 0))
+      (scale (xyz 1 1 1))
+      (rotate (xyz 0 0 0))
+    )
+  )
   (gr_line (start -8.89 8.89) (end -8.89 -8.89) (angle 90) (layer Edge.Cuts) (width 0.15))
   (gr_line (start 8.89 8.89) (end -8.89 8.89) (angle 90) (layer Edge.Cuts) (width 0.15))
@@
   (segment (start -7.34822 -6.35) (end -6.096 -4.699) (width 0.25) (layer B.Cu) (net 4) (status 10))
   (segment (start -6.096 -4.699) (end -3.81 -2.54) (width 0.25) (layer B.Cu) (net 4) (status 20))
+  (segment (start 1.04902 3.175) (end 1.04902 3.175) (width 0.25) (layer B.Cu) (net 5) (status C00000))
+  (segment (start 1.04902 3.175) (end 3.81 5.08) (width 0.25) (layer B.Cu) (net 5) (status C00000))
   (segment (start 3.81 5.08) (end 7.62 2.54) (width 0.25) (layer B.Cu) (net 5) (status 30))
+  (segment (start -1.04902 3.175) (end -1.04902 3.175) (width 0.25) (layer B.Cu) (net 6) (status C00000))
+  (segment (start -1.04902 3.175) (end -3.81 5.08) (width 0.25) (layer B.Cu) (net 6) (status C00000))
   (segment (start -3.81 5.08) (end -1.523859 6.172174) (width 0.25) (layer F.Cu) (net 6) (status 10))
   (segment (start 3.936807 6.18731) (end 7.62 5.08) (width 0.25) (layer F.Cu) (net 6) (status 20))
   (segment (start -1.523859 6.172174) (end 3.936807 6.18731) (width 0.25) (layer F.Cu) (net 6))
-  (segment (start 1.27 5.08) (end 7.62 0) (width 0.25) (layer B.Cu) (net 7) (status 30))
+  (segment (start 1.27 5.08) (end 7.62 0) (width 0.25) (layer F.Cu) (net 7) (status C00000))
+  (segment (start 7.62 0) (end 7.62 0) (width 0.25) (layer F.Cu) (net 7) (status C00000))
+  (segment (start 7.62 0) (end 7.62 0) (width 0.25) (layer F.Cu) (net 7) (status C00000))
+  (segment (start 7.62 0) (end 7.62 0) (width 0.25) (layer F.Cu) (net 7) (status C00000))
   (segment (start -1.27 5.08) (end 0.856873 6.15931) (width 0.25) (layer B.Cu) (net 8) (status 10))
   (segment (start 0.856873 6.15931) (end 7.62 7.62) (width 0.25) (layer B.Cu) (net 8) (status 20))
