File: LED-Driver/LED-Driver.kicad_pcb (KiCad board)
At the start: 2 copper layers, 40.6 x 22.9 mm, 27 parts, among them P1 CONN_02X04, P2 CONN_02X04, P3 CONN_01X05, P4 CONN_01X02, P5 CONN_01X09, P6 CONN_01X09, U1 IS31FL3732

Commit message: Switched to 2.5mm Mounting Holes
Parts:
- removed the ? at (576.6, 416.6)
- removed the ? at (617.2, 414.0)
- removed the ? at (576.6, 403.9)
- removed the ? at (617.2, 405.1)
- added ?: MountingHole_2.5mm, Mounting_Holes:MountingHole_2.5mm, F.Cu at (576.6, 403.9)
- added ?: MountingHole_2.5mm, Mounting_Holes:MountingHole_2.5mm, F.Cu at (576.6, 416.6)
- added ?: MountingHole_2.5mm, Mounting_Holes:MountingHole_2.5mm, F.Cu at (617.2, 414.0)
- added ?: MountingHole_2.5mm, Mounting_Holes:MountingHole_2.5mm, F.Cu at (617.2, 405.1)
Routing:
- net (no net): track 0.00 -> 1.53 mm

Commit message: Minor cleanups
Routing:
- net (no net): track 1.53 -> 0.00 mm
