File: Chain-Connector/Chain-Connector.sch (KiCad schematic (older format))
At the start: 7 parts, among them P1 USB_A, P2 CONN_01X06, U1 SN74HC157PWR

Commit message: Added the Option to use a Micro-USB Connector
And also revamped the Routing to be less of a Mess
Parts:
- added P3: USB_OTG, Connect:USB_Micro-B, symbol USB_OTG
Connections:
- wire segments 35 -> 39
- no-connect marks 2 -> 4
Other:
- moved on the sheet: D3, P1, P2, R1
Changed lines of the file:
@@
 L USB_A P1
 U 1 1 57226042
-P 2250 1550
-F 0 "P1" H 2450 1350 50  0000 C CNN
-F 1 "USB_A" H 2200 1750 50  0000 C CNN
-F 2 "Connect:USB_A" V 2200 1450 50  0001 C CNN
-F 3 "" V 2200 1450 50  0000 C CNN
-	1    2250 1550
+P 2250 950
+F 0 "P1" H 2450 750 50  0000 C CNN
+F 1 "USB_A" H 2200 1150 50  0000 C CNN
+F 2 "Connect:USB_A" V 2200 850 50  0001 C CNN
+F 3 "" V 2200 850 50  0000 C CNN
+	1    2250 950
 	0    1    1    0
 $EndComp
-NoConn ~ 2350 1850
-Wire Wire Line
-	1950 1350 1850 1350
-Wire Wire Line
-	1950 1450 1850 1450
-Wire Wire Line
-	1950 1550 1850 1550
-Wire Wire Line
-	1950 1650 1850 1650
-Wire Wire Line
-	2050 2050 1850 2050
-Wire Wire Line
-	2050 2150 1850 2150
-Wire Wire Line
-	1750 2250 2050 2250
+NoConn ~ 2350 1250
+Wire Wire Line
+	1950 750  1850 750
+Wire Wire Line
+	1950 850  1850 850
+Wire Wire Line
+	1950 950  1850 950
+Wire Wire Line
+	1950 1050 1850 1050
 Wire Wire Line
 	2050 2350 1850 2350
-Text Label 1850 1450 2    60   ~ 0
+Wire Wire Line
+	2050 2450 1850 2450
+Wire Wire Line
+	1750 2550 2050 2550
+Wire Wire Line
+	2050 2650 1850 2650
+Text Label 1850 850  2    60   ~ 0
 IO1
-Text Label 1850 1550 2    60   ~ 0
+Text Label 1850 950  2    60   ~ 0
 IO2
-Text Label 1850 2350 2    60   ~ 0
+Text Label 1850 2650 2    60   ~ 0
 TX0
-Text Label 1850 2150 2    60   ~ 0
+Text Label 1850 2450 2    60   ~ 0
 RX0
 $Comp
 L CONN_01X06 P2
 U 1 1 57236A8A
-P 2250 2300
-F 0 "P2" H 2250 2650 50  0000 C CNN
-F 1 "CONN_01X06" V 2350 2300 50  0000 C CNN
-F 2 "Pin_Headers:Pin_Header_Straight_2x03" H 2250 2300 50  0001 C CNN
-F 3 "" H 2250 2300 50  0000 C CNN
-	1    2250 2300
-	1    0    0    -1
-$EndComp
-Wire Wire Line
-	2050 2450 1850 2450
-Text Label 1850 2450 2    60   ~ 0
+P 2250 2600
+F 0 "P2" H 2250 2950 50  0000 C CNN
+F 1 "CONN_01X06" V 2350 2600 50  0000 C CNN
+F 2 "Pin_Headers:Pin_Header_Straight_2x03" H 2250 2600 50  0001 C CNN
+F 3 "" H 2250 2600 50  0000 C CNN
+	1    2250 2600
+	1    0    0    -1
+$EndComp
+Wire Wire Line
+	2050 2750 1850 2750
+Text Label 1850 2750 2    60   ~ 0
 Master
-NoConn ~ 2050 2550
+NoConn ~ 2050 2850
 $Comp
 L LED D3
 U 1 1 57237083
-P 2250 2800
-F 0 "D3" H 2250 2900 50  0000 C CNN
-F 1 "LED" H 2250 2700 50  0000 C CNN
-F 2 "LEDs:LED_0805" H 2250 2800 50  0001 C CNN
-F 3 "" H 2250 2800 50  0000 C CNN
-	1    2250 2800
-	-1   0    0    1
-$EndComp
-Text Label 1850 2800 2    60   ~ 0
+P 2250 3150
+F 0 "D3" H 2250 3250 50  0000 C CNN
+F 1 "LED" H 2250 3050 50  0000 C CNN
+F 2 "LEDs:LED_0805" H 2250 3150 50  0001 C CNN
+F 3 "" H 2250 3150 50  0000 C CNN
+	1    2250 3150
+	-1   0    0    1
+$EndComp
+Text Label 1850 3150 2    60   ~ 0
 Master
 Wire Wire Line
-	2050 2800 1850 2800
+	2050 3150 1850 3150
 $Comp
 L R R1
 U 1 1 572372DF
-P 2600 2800
-F 0 "R1" V 2680 2800 50  0000 C CNN
-F 1 "1k" V 2600 2800 50  0000 C CNN
-F 2 "Resistors_SMD:R_0603" V 2530 2800 50  0001 C CNN
-F 3 "" H 2600 2800 50  0000 C CNN
-	1    2600 2800
+P 2600 3150
+F 0 "R1" V 2680 3150 50  0000 C CNN
+F 1 "1k" V 2600 3150 50  0000 C CNN
+F 2 "Resistors_SMD:R_0603" V 2530 3150 50  0001 C CNN
+F 3 "" H 2600 3150 50  0000 C CNN
+	1    2600 3150
 	0    1    1    0
 $EndComp
 Wire Wire Line
-	2750 2800 2850 2800
-Wire Wire Line
-	2850 2800 2850 2900
+	2750 3150 2850 3150
+Wire Wire Line
+	2850 3150 2850 3250
 $Comp
 L VCC #PWR01
 U 1 1 572374C1
-P 1850 1350
-F 0 "#PWR01" H 1850 1200 50  0001 C CNN
-F 1 "VCC" H 1850 1500 50  0000 C CNN
-F 2 "" H 1850 1350 50  0000 C CNN
-F 3 "" H 1850 1350 50  0000 C CNN
-	1    1850 1350
+P 1850 750
+F 0 "#PWR01" H 1850 600 50  0001 C CNN
+F 1 "VCC" H 1850 900 50  0000 C CNN
+F 2 "" H 1850 750 50  0000 C CNN
+F 3 "" H 1850 750 50  0000 C CNN
+	1    1850 750
 	1    0    0    -1
 $EndComp
@@
 L VCC #PWR02
 U 1 1 5723750F
-P 1750 2250
-F 0 "#PWR02" H 1750 2100 50  0001 C CNN
-F 1 "VCC" H 1750 2400 50  0000 C CNN
-F 2 "" H 1750 2250 50  0000 C CNN
-F 3 "" H 1750 2250 50  0000 C CNN
-	1    1750 2250
+P 1750 2550
+F 0 "#PWR02" H 1750 2400 50  0001 C CNN
+F 1 "VCC" H 1750 2700 50  0000 C CNN
+F 2 "" H 1750 2550 50  0000 C CNN
+F 3 "" H 1750 2550 50  0000 C CNN
+	1    1750 2550
 	0    -1   -1   0
 $EndComp
@@
 L GND #PWR03
 U 1 1 57237864
-P 1850 1650
-F 0 "#PWR03" H 1850 1400 50  0001 C CNN
-F 1 "GND" H 1850 1500 50  0000 C CNN
-F 2 "" H 1850 1650 50  0000 C CNN
-F 3 "" H 1850 1650 50  0000 C CNN
-	1    1850 1650
+P 1850 1050
+F 0 "#PWR03" H 1850 800 50  0001 C CNN
+F 1 "GND" H 1850 900 50  0000 C CNN
+F 2 "" H 1850 1050 50  0000 C CNN
+F 3 "" H 1850 1050 50  0000 C CNN
+	1    1850 1050
 	1    0    0    -1
 $EndComp
@@
 L GND #PWR04
 U 1 1 57237882
-P 1850 2050
-F 0 "#PWR04" H 1850 1800 50  0001 C CNN
-F 1 "GND" H 1850 1900 50  0000 C CNN
-F 2 "" H 1850 2050 50  0000 C CNN
-F 3 "" H 1850 2050 50  0000 C CNN
-	1    1850 2050
+P 1850 2350
+F 0 "#PWR04" H 1850 2100 50  0001 C CNN
+F 1 "GND" H 1850 2200 50  0000 C CNN
+F 2 "" H 1850 2350 50  0000 C CNN
+F 3 "" H 1850 2350 50  0000 C CNN
+	1    1850 2350
 	-1   0    0    1
 $EndComp
@@
 L GND #PWR05
 U 1 1 5723791D
-P 2850 2900
-F 0 "#PWR05" H 2850 2650 50  0001 C CNN
-F 1 "GND" H 2850 2750 50  0000 C CNN
-F 2 "" H 2850 2900 50  0000 C CNN
-F 3 "" H 2850 2900 50  0000 C CNN
-	1    2850 2900
+P 2850 3250
+F 0 "#PWR05" H 2850 3000 50  0001 C CNN
+F 1 "GND" H 2850 3100 50  0000 C CNN
+F 2 "" H 2850 3250 50  0000 C CNN
+F 3 "" H 2850 3250 50  0000 C CNN
+	1    2850 3250
 	1    0    0    -1
 $EndComp
@@
 	4850 2200 5250 2200
 Connection ~ 5250 2200
+$Comp
+L USB_OTG P3
+U 1 1 574B1B1F
+P 2250 1700
+F 0 "P3" H 2575 1575 50  0000 C CNN
+F 1 "USB_OTG" H 2250 1900 50  0000 C CNN
+F 2 "Connect:USB_Micro-B" V 2200 1600 50  0001 C CNN
+F 3 "" V 2200 1600 50  0000 C CNN
+	1    2250 1700
+	0    1    1    0
+$EndComp
+NoConn ~ 2350 2100
+Wire Wire Line
+	1950 1500 1850 1500
+Wire Wire Line
+	1950 1600 1850 1600
+Wire Wire Line
+	1950 1700 1850 1700
+Wire Wire Line
+	1950 1900 1850 1900
+Text Label 1850 1600 2    60   ~ 0
+IO1
+Text Label 1850 1700 2    60   ~ 0
+IO2
+$Comp
+L VCC #PWR011
+U 1 1 574B1BCE
+P 1850 1500
+F 0 "#PWR011" H 1850 1350 50  0001 C CNN
+F 1 "VCC" H 1850 1650 50  0000 C CNN
+F 2 "" H 1850 1500 50  0000 C CNN
+F 3 "" H 1850 1500 50  0000 C CNN
+	1    1850 1500
+	1    0    0    -1
+$EndComp
+$Comp
+L GND #PWR012
+U 1 1 574B1BD4
+P 1850 1900
+F 0 "#PWR012" H 1850 1650 50  0001 C CNN
+F 1 "GND" H 1850 1750 50  0000 C CNN
+F 2 "" H 1850 1900 50  0000 C CNN
+F 3 "" H 1850 1900 50  0000 C CNN
+	1    1850 1900
+	1    0    0    -1
+$EndComp
+NoConn ~ 1950 1800
 $EndSCHEMATC
